Commit message: 1.changed ik and myrobot_descriptioin launch file to communicate with ROS 2. changed RVIZ model to comply with our current default position and new locomotion design

File: catkin_ws/src/myrobot_description/urdf/robot_cali.urdf (robot description, URDF)
Before this commit: robot TheBoatDoctor, 9 links, 8 joints
Joints:
- joint joint_world_locomotion: origin xyz=0 0 0.1464 rpy=0 0 1.57 -> xyz=0 0 0.1718 rpy=0 0 1.57
